File: pcb/pic18_edd.kicad_pcb (KiCad board)
At the start: 2 copper layers, 77.5 x 67.6 mm, 51 parts, among them IC1 MIKROE-2439, J1 Conn_UART, J2 Conn_BAT, J3 Conn_CAN, J4 Conn_PROG, J5 Conn_MOTOR, K1 SR5-12V-200-1C, Q1 BC817-25-QR, SW1 SW_reset, SW2 SW_2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

Commit message: last version
Parts:
- removed SW3: SW_3, Components:Push_btn_SMD
- added SW0: SW_reset, Components:Push_btn_SMD_sqr_handsoldering, F.Cu at (123.5, 83.9)
- D3: footprint Diode_SMD:D_SMF -> Diode_SMD:D_SMA_Handsoldering
- D5: value 156120VS75000 Red -> 156120RS75000 Red
- FB1: footprint Inductor_SMD:L_Ferrocore_DLG-0302 -> Inductor_SMD:L_0402_1005Metric_Pad0.77x0.64mm_HandSolder
- SW1: value SW_reset -> SW_1; footprint Components:Push_btn_SMD -> Components:Push_btn_SMD_sqr_handsoldering
- SW2: footprint Components:Push_btn_SMD -> Components:Push_btn_SMD_sqr_handsoldering
- U4: footprint Package_SO:SSOP-28_5.3x10.2mm_P0.65mm -> Package_SO:SOIC-28W_7.5x18.7mm_P1.27mm
- moved SW1 16.7 mm to (123.5, 67.3)
- moved SW2 8.64 mm to (123.5, 75.5)
- moved C5 8.04 mm to (161.5, 75.4)
- moved R10 4.89 mm to (168.9, 77.5)
- moved R11 4.79 mm to (168.9, 73.8)
- moved C7 4.48 mm to (141.2, 86.1)
- moved C8 4.18 mm to (183.8, 75.4)
- moved U5 4.18 mm to (177.8, 75.5)
- moved U3 4.18 mm to (151.1, 84.8)
- moved U4 3.17 mm to (148.6, 75.8)
- moved R7 3.12 mm to (131.4, 84.1)
- moved R5 3.12 mm to (131.4, 75.9)
- moved R6 2.76 mm to (131.4, 67.7)
- moved D4 1.34 mm to (121.4, 61.7)
- moved D5 1.34 mm to (121.4, 57.5)
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Connections:
- SW1 pad 3: VPP_MCLR -> INPUT_1
- SW2 pad 3: INPUT_1 -> INPUT_2
Routing:
- net INPUT_1: track 19.8 -> 27.1 mm
- net MOTOR_H: track 12.6 -> 6.28 mm
- net U_TX: track 54.0 -> 49.2 mm
- net INPUT_2: track 17.3 -> 22.1 mm
- net VPP_MCLR: track 60.0 -> 55.3 mm
- net I2C_DATA: track 44.5 -> 40.0 mm
- net U_RX: track 45.4 -> 41.4 mm
- net I2C_CLK: track 46.0 -> 43.4 mm
- net Net-(U4-Vcap): track 6.84 -> 9.43 mm
- net /LED_R: track 24.6 -> 26.8 mm
- net /LED_G: track 26.7 -> 28.3 mm
- net CAN_TX: track 10.2 -> 11.6 mm
- net Net-(D6-A): track 2.18 -> 3.52 mm
- net Net-(D5-A): track 2.18 -> 3.52 mm
- net Net-(D4-A): track 2.18 -> 3.52 mm
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Other:
- board text added: "MIKROE socket"
- board text removed: "MIKRO E2439"
- board text removed: "module"
