File: pcb/pic18_edd.kicad_sch (KiCad schematic)
At the start: 51 parts, among them IC1 MIKROE-2439, J1 Conn_UART, J2 Conn_BAT, J3 Conn_CAN, J4 Conn_PROG, J5 Conn_MOTOR, K1 SR5-12V-200-1C, Q1 BC817-25-QR, SW1 SW_reset, SW2 SW_2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

Commit message: last version
Parts:
- D3: footprint Diode_SMD:D_SMF -> Diode_SMD:D_SMA_Handsoldering
- D5: value 156120VS75000 Red -> 156120RS75000 Red
- FB1: footprint Inductor_SMD:L_Ferrocore_DLG-0302 -> Inductor_SMD:L_0402_1005Metric_Pad0.77x0.64mm_HandSolder
- SW0: renamed from SW1; footprint Components:Push_btn_SMD -> Components:Push_btn_SMD_sqr_handsoldering
- SW1: renamed from SW2; value SW_2 -> SW_1; footprint Components:Push_btn_SMD -> Components:Push_btn_SMD_sqr_handsoldering
- SW2: renamed from SW3; value SW_3 -> SW_2; footprint Components:Push_btn_SMD -> Components:Push_btn_SMD_sqr_handsoldering
- U4: footprint Package_SO:SSOP-28_5.3x10.2mm_P0.65mm -> Package_SO:SOIC-28W_7.5x18.7mm_P1.27mm
Changed lines of the file:
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@@
       (effects (font (size 1.27 1.27)))
     )
-    (property "Footprint" "Package_SO:SSOP-28_5.3x10.2mm_P0.65mm" (at 111.252 108.966 0)
+    (property "Footprint" "Package_SO:SOIC-28W_7.5x18.7mm_P1.27mm" (at 111.252 108.966 0)
       (effects (font (size 1.27 1.27)) hide)
     )
@@
       (effects (font (size 1.27 1.27)) (justify left))
     )
-    (property "Footprint" "Inductor_SMD:L_Ferrocore_DLG-0302" (at 38.608 41.91 90)
+    (property "Footprint" "Inductor_SMD:L_0402_1005Metric_Pad0.77x0.64mm_HandSolder" (at 38.608 41.91 90)
       (effects (font (size 1.27 1.27)) hide)
     )
@@
   (symbol (lib_id "Components:SW_Push_Single") (at 225.298 101.346 0) (unit 1)
     (in_bom yes) (on_board yes) (dnp no) (fields_autoplaced)
-    (property "Reference" "SW2" (at 231.14 103.759 0)
-      (effects (font (size 1.27 1.27)) (justify left))
-    )
-    (property "Value" "SW_2" (at 231.14 106.299 0)
-      (effects (font (size 1.27 1.27)) (justify left))
-    )
-    (property "Footprint" "Components:Push_btn_SMD" (at 233.299 104.267 90)
+    (property "Reference" "SW1" (at 231.14 103.759 0)
+      (effects (font (size 1.27 1.27)) (justify left))
+    )
+    (property "Value" "SW_1" (at 231.14 106.299 0)
+      (effects (font (size 1.27 1.27)) (justify left))
+    )
+    (property "Footprint" "Components:Push_btn_SMD_sqr_handsoldering" (at 233.299 104.267 90)
       (effects (font (size 1.27 1.27)) hide)
     )
@@
       (project "pic18_edd"
         (path "/e5a7d9d1-7845-4bdc-8658-31f5022a919f"
-          (reference "SW2") (unit 1)
+          (reference "SW1") (unit 1)
         )
       )
@@
   (symbol (lib_id "Components:SW_Push_Single") (at 196.85 101.6 0) (unit 1)
     (in_bom yes) (on_board yes) (dnp no) (fields_autoplaced)
-    (property "Reference" "SW1" (at 203.2 104.013 0)
+    (property "Reference" "SW0" (at 203.2 104.013 0)
       (effects (font (size 1.27 1.27)) (justify left))
     )
@@
       (effects (font (size 1.27 1.27)) (justify left))
     )
-    (property "Footprint" "Components:Push_btn_SMD" (at 204.851 104.521 90)
+    (property "Footprint" "Components:Push_btn_SMD_sqr_handsoldering" (at 204.851 104.521 90)
       (effects (font (size 1.27 1.27)) hide)
     )
@@
       (project "pic18_edd"
         (path "/e5a7d9d1-7845-4bdc-8658-31f5022a919f"
-          (reference "SW1") (unit 1)
+          (reference "SW0") (unit 1)
         )
       )
@@
       (effects (font (size 1.27 1.27)) (justify left))
     )
-    (property "Footprint" "Diode_SMD:D_SMF" (at 69.596 39.878 0)
+    (property "Footprint" "Diode_SMD:D_SMA_Handsoldering" (at 69.596 39.878 0)
       (effects (font (size 1.27 1.27)) hide)
     )
@@
       (effects (font (size 1.27 1.27)) (justify right))
     )
-    (property "Value" "156120VS75000 Red" (at 161.036 99.06 0)
+    (property "Value" "156120RS75000 Red" (at 161.036 99.06 0)
       (effects (font (size 1.27 1.27)) (justify right))
     )
@@
   (symbol (lib_id "Components:SW_Push_Single") (at 254 101.6 0) (unit 1)
     (in_bom yes) (on_board yes) (dnp no) (fields_autoplaced)
-    (property "Reference" "SW3" (at 260.35 104.013 0)
-      (effects (font (size 1.27 1.27)) (justify left))
-    )
-    (property "Value" "SW_3" (at 260.35 106.553 0)
-      (effects (font (size 1.27 1.27)) (justify left))
-    )
-    (property "Footprint" "Components:Push_btn_SMD" (at 262.001 104.521 90)
+    (property "Reference" "SW2" (at 260.35 104.013 0)
+      (effects (font (size 1.27 1.27)) (justify left))
+    )
+    (property "Value" "SW_2" (at 260.35 106.553 0)
+      (effects (font (size 1.27 1.27)) (justify left))
+    )
+    (property "Footprint" "Components:Push_btn_SMD_sqr_handsoldering" (at 262.001 104.521 90)
       (effects (font (size 1.27 1.27)) hide)
     )
@@
       (project "pic18_edd"
         (path "/e5a7d9d1-7845-4bdc-8658-31f5022a919f"
-          (reference "SW3") (unit 1)
-        )
-      )
+          (reference "SW2") (unit 1)
+        )
+      )
